File: PCB/HostBoard/HostBoard_DoubleGND.kicad_pcb (KiCad board)
At the start: 4 copper layers, 52 x 77.5 mm, 23 parts, among them J1 Conn_01x06, J10 Conn_01x05, J11 Screw_Terminal_01x02, J12 Conn_02x07_Odd_Even, J2 Conn_01x03, J3 Conn_01x06, J4 Conn_01x03, J5 Conn_01x06, J6 Conn_01x04, J7 Conn_01x04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

Commit message: As sent to JLBPCB. $66.
Parts:
- added J13: Conn_01x02, Connector_PinHeader_2.54mm:PinHeader_1x02_P2.54mm_Vertical, F.Cu at (70.8, 113.4)
- added TP2: 5V, Connector_PinHeader_2.54mm:PinHeader_1x01_P2.54mm_Vertical, F.Cu at (84.7, 51.7)
- added TP5: 3V3, Connector_PinHeader_2.54mm:PinHeader_1x01_P2.54mm_Vertical, F.Cu at (90.1, 51.7)
- added TP6: CL_A, TestPoint:TestPoint_Pad_1.0x1.0mm, B.Cu at (71.3, 80.7)
- added TP7: CL_B, TestPoint:TestPoint_Pad_1.0x1.0mm, B.Cu at (69.8, 83.6)
- TP1: value TestPoint -> SD_DC
- moved J11 0.96 mm to (53.7, 120.6)
Connections:
- net /SD_CD renamed /SD_DC
- A1 pad 19: unconnected-(A1-GPIO14-Pad19) -> /GP14
- A1 pad 20: unconnected-(A1-GPIO15-Pad20) -> /GP15
- A1 pad 33: unconnected-(A1-AGND-Pad33) -> GND
- U1 pad 7: unconnected-(U1-GPB6-Pad7) -> /COMPASS_LIMIT_A
- U1 pad 8: unconnected-(U1-GPB7-Pad8) -> /COMPASS_LIMIT_B
- U2 pad 11: Net-(J3-Pin_1) -> Net-(J3-Pin_6)
- U2 pad 12: Net-(J3-Pin_1) -> Net-(J3-Pin_6)
- U2 pad 7: Net-(J3-Pin_6) -> Net-(J3-Pin_1)
- U2 pad 8: Net-(J3-Pin_6) -> Net-(J3-Pin_1)
Routing:
- net +3.3V: track 284.2 -> 358.4 mm
- net /GP14: track 0.00 -> 19.8 mm
- net /GP15: track 0.00 -> 15.0 mm
- net /COMPASS_LIMIT_A: track 0.00 -> 13.7 mm
- net /COMPASS_LIMIT_B: track 0.00 -> 13.4 mm, vias 0 -> 2
- net Net-(J3-Pin_6): track 40.1 -> 33.2 mm, vias 3 -> 2
- net GND: track 46.0 -> 52.0 mm
- net Net-(J1-Pin_6): track 37.0 -> 41.9 mm
- net Net-(J3-Pin_1): track 48.0 -> 52.7 mm
- net +5V: track 87.8 -> 92.1 mm
- net Net-(J5-Pin_6): track 27.2 -> 30.5 mm, vias 2 -> 0
- net Vmotor: track 136.6 -> 134.2 mm
- net SCL_0: track 126.7 -> 124.5 mm
- net SDA_0: track 122.2 -> 120.6 mm
Other:
- board text added: "3V3"
- board text added: "5V"
- board text added: "A"
- board text added: "A1 - Raspberry Pi Pico 2 W U1 - MCP23017SS I/O Expander U2, U3 - TB6612FNG DC Motor Drive"
- board text added: "B"
- board text added: "GP14"
- board text added: "GP15"
- board text added: "McA ©2025"
- board text added: "N/C"
- board text added: "SD_DC"
- board text added: "SPARE MOT"
- board text added: "XY Tracker DC MOTOR / CONTROL"
- board text removed: "SD_CD"
